File: Pistachio_MacroPad/Pistachio_MacroPad.kicad_pcb (KiCad board)
At the start: 2 copper layers, 86.1 x 133.7 mm, 53 parts, among them J2 Conn_01x02, SW1 SW_Push, SW10 SW_Push, SW11 SW_Push, SW12 SW_Push, SW13 SW_Push, SW14 SW_Push, SW15 SW_Push, SW16 SW_Push, SW17 SW_Push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

Commit message: v1.1
Parts:
- removed Je: AudioJack4, keyboard:MJ-4PP-9_1side
- added BT1: Battery_Cell, keyboard:BAT_HLD-001, F.Cu at (156.7, 33.3)
- added G***: LOGO, logo:pistachio_name, B.Cu at (142.9, 146.9)
- added G***: LOGO, logo:pistachio_log, B.Cu at (178.5, 139.9)
- added J1: AudioJack4, keyboard:MJ-4PP-9_1side, B.Cu at (35.2, 24.9)
- added J3: Conn_01x02, keyboard:POWER_PAD, F.Cu at (191.8, 81.7)
- added SW20: SW_DIP_x01, keyboard:SlideSwitch_IS-2245S-G, F.Cu at (175.0, 27.1)
- moved R4 52.7 mm to (34.5, 38.3), turned to 180 degrees
- moved R3 48.8 mm to (30.7, 34.3)
- moved U1 4.55 mm to (48.4, 43.2)
- moved J2 0.69 mm to (109.9, 59.9)
- turned SW12 to 90 degrees
- turned SW18 to 90 degrees
Routing:
- net Net-(BT1-Pad2): track 0.00 -> 103.0 mm
- net Net-(J3-Pad1): track 0.00 -> 65.3 mm
- net GND: track 225.6 -> 161.1 mm, vias 1 -> 97
- net Net-(BT1-Pad1): track 0.00 -> 48.9 mm
- net SDA: track 55.7 -> 7.95 mm
- net SCL: track 57.1 -> 31.6 mm
- net Net-(D12-Pad1): track 22.0 -> 28.6 mm
- net col3: track 209.7 -> 203.6 mm
- net Net-(D18-Pad1): track 22.9 -> 28.6 mm
- net encB: track 69.3 -> 63.9 mm
- net encA: track 69.0 -> 63.6 mm
- net BAT: track 89.9 -> 85.2 mm
- net col2: track 220.9 -> 216.2 mm
- net reset: track 81.9 -> 77.9 mm
- net col0: track 203.6 -> 206.8 mm
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- added copper zone on B.Cu, net GND
- added copper zone on F.Cu, net GND
Other:
- board size 86.1 x 133.7 mm -> 173.3 x 133.7 mm
- board text added: "Designed by 7_rate"
- board text added: "Don't implement D20 when closing JP1"
- board text added: "OFF"
- board text added: "ON"
- board text added: "PistachioMacroPad_v1.1"
