File: Pistachio_MacroPad/Pistachio_MacroPad.sch (KiCad schematic (older format))
At the start: 50 parts, among them J1 AudioJack4, J2 Conn_01x02, SW1 SW_Push, SW10 SW_Push, SW11 SW_Push, SW12 SW_Push, SW13 SW_Push, SW14 SW_Push, SW15 SW_Push, SW16 SW_Push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

Commit message: v1.1
Parts:
- added BT1: Battery_Cell, keyboard:BAT_HLD-001, symbol Device:Battery_Cell
- added J3: Conn_01x02, keyboard:POWER_PAD, symbol Connector_Generic:Conn_01x02
- added SW20: SW_DIP_x01, keyboard:SlideSwitch_IS-2245S-G, symbol Switch:SW_DIP_x01
Connections:
- new net: BT1.1 (+), SW20.1
- new net: J3.1 (Pin_1), SW20.2
- new net: BT1.2 (-), J3.2 (Pin_2)
Changed lines of the file:
@@
 Text GLabel 7700 1250 2    50   Output ~ 0
 encB
+$Comp
+L Switch:SW_DIP_x01 SW20
+U 1 1 5F9AE7A9
+P 1500 6750
+F 0 "SW20" H 1500 7017 50  0000 C CNN
+F 1 "SW_DIP_x01" H 1500 6926 50  0000 C CNN
+F 2 "keyboard:SlideSwitch_IS-2245S-G" H 1500 6750 50  0001 C CNN
+F 3 "~" H 1500 6750 50  0001 C CNN
+	1    1500 6750
+	1    0    0    -1
+$EndComp
+$Comp
+L Device:Battery_Cell BT1
+U 1 1 5F9AFEEC
+P 950 7100
+F 0 "BT1" H 1068 7196 50  0000 L CNN
+F 1 "Battery_Cell" H 1068 7105 50  0000 L CNN
+F 2 "keyboard:BAT_HLD-001" V 950 7160 50  0001 C CNN
+F 3 "~" V 950 7160 50  0001 C CNN
+	1    950  7100
+	1    0    0    -1
+$EndComp
+$Comp
+L Connector_Generic:Conn_01x02 J3
+U 1 1 5F9B0936
+P 2150 7000
+F 0 "J3" H 2230 6992 50  0000 L CNN
+F 1 "Conn_01x02" H 2230 6901 50  0000 L CNN
+F 2 "keyboard:POWER_PAD" H 2150 7000 50  0001 C CNN
+F 3 "~" H 2150 7000 50  0001 C CNN
+	1    2150 7000
+	1    0    0    -1
+$EndComp
+$Comp
+L power:PWR_FLAG #FLG03
+U 1 1 5F9B1993
+P 950 6750
+F 0 "#FLG03" H 950 6825 50  0001 C CNN
+F 1 "PWR_FLAG" H 950 6923 50  0000 C CNN
+F 2 "" H 950 6750 50  0001 C CNN
+F 3 "~" H 950 6750 50  0001 C CNN
+	1    950  6750
+	1    0    0    -1
+$EndComp
+Wire Wire Line
+	950  6900 950  6750
+Wire Wire Line
+	950  6750 1200 6750
+Wire Wire Line
+	1800 6750 1950 6750
+Wire Wire Line
+	1950 6750 1950 7000
+Wire Wire Line
+	1950 7100 1950 7300
+Wire Wire Line
+	1950 7300 950  7300
+Wire Wire Line
+	950  7300 950  7200
+Connection ~ 950  6750
+$Comp
+L power:PWR_FLAG #FLG04
+U 1 1 5F9BA88A
+P 950 7300
+F 0 "#FLG04" H 950 7375 50  0001 C CNN
+F 1 "PWR_FLAG" H 950 7473 50  0000 C CNN
+F 2 "" H 950 7300 50  0001 C CNN
+F 3 "~" H 950 7300 50  0001 C CNN
+	1    950  7300
+	-1   0    0    1
+$EndComp
+Connection ~ 950  7300
 $EndSCHEMATC
