File: Pistachio_MacroPad_rev1.0/Pistachio_MacroPad.sch (KiCad schematic (older format))
At the start: 53 parts, among them J1 AudioJack4, J2 Conn_01x02, J3 Conn_01x02, SW1 SW_Push, SW10 SW_Push, SW11 SW_Push, SW12 SW_Push, SW13 SW_Push, SW14 SW_Push, SW15 SW_Push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

Commit message: フォルダ構造整理
Parts:
- BT1: footprint keyboard:BAT_HLD-001 -> kbd:BAT_HLD-001
- D1, D10, D11, D12, D13, D14, D15, D16, D17, D18, D2, D3, D4, D5, D6, D7, D8, D9: footprint keyboard:D3_SMD_v2 -> kbd:D3_SMD_v2
- D19, D20, D21: footprint keyboard:WS2812C-2020 -> kbd:WS2812C-2020; symbol keyboard:WS2812C -> kbd:WS2812C
- J1: footprint keyboard:MJ-4PP-9_1side -> kbd:MJ-4PP-9_1side
- J2: footprint keyboard:S2B-ZR-3.4 -> kbd:S2B-ZR-3.4
- J3: footprint keyboard:POWER_PAD -> kbd:POWER_PAD
- SW1, SW10, SW11, SW12, SW13, SW14, SW15, SW16, SW17, SW18, SW2, SW3, SW4, SW5, SW6, SW7, SW9: footprint keyswitches:Kailh_socket_MX_optional -> kbd:Kailh_socket_MX_optional
- SW19: footprint keyboard:ResetSW_1side -> kbd:ResetSW_1side
- SW20: footprint keyboard:SlideSwitch_IS-2245S-G -> kbd:SlideSwitch_IS-2245S-G
- SW8: footprint keyboard:PEC12R-4xxxF-Sxxxx -> kbd:PEC12R-4xxxF-Sxxxx
- U1: footprint keyboard:ProMicro_BLE -> kbd:ProMicro_BLE; symbol keyboard:BLE_Micro_Pro -> kbd:BLE_Micro_Pro
